File: pcb/aeroportal.kicad_sch (KiCad schematic)
At the start: 4 parts, among them J1 MAX98357A Breakout Board, U1 WEMOS_C3_Mini, U2 TFT_ST7735_SD

Commit message: Created basic firmware and fixed unconnected pin for speaker
Signed-off-by: Urjith Mishra <66270347+TheScientist101@users.noreply.github.com>
Connections:
- net LRC: now also U1.2 (IO3)
Changed lines of the file:
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@@
+		)
+	)
+	(global_label "LRC"
+		(shape input)
+		(at 106.68 62.23 0)
+		(fields_autoplaced yes)
+		(effects
+			(font
+				(size 1.27 1.27)
+			)
+			(justify left)
+		)
+		(property "Intersheetrefs" "${INTERSHEET_REFS}"
+			(at 113.2333 62.23 0)
+			(effects
+				(font
+					(size 1.27 1.27)
+				)
+				(justify left)
+				(hide yes)
+			)
 		)
 	)
